Commit message: Fix robot model: geometry, Gazebo materials, ParameterValue wrapping
- Wrap xacro output in ParameterValue for Humble compatibility
- Add Gazebo material colors (FlatBlack, Orange, Blue, Grey)
- Add top plate, front bumper, sensor tower links
- Fix drive wheel z-offset so wheels touch ground
- Fix caster wheel geometry (larger radius, correct z-offset)
- Correct wheel_separation to match actual URDF geometry

File: src/amr_description/urdf/amr.urdf.xacro (robot description, xacro)
@@ -1,5 +1,5 @@
 <?xml version="1.0"?>
 <robot xmlns:xacro="http://www.ros.org/wiki/xacro" name="amr">
-  <!-- ==================== Material Definitions ==================== -->
+  <!-- ==================== Material Definitions (RViz) ==================== -->
   <material name="dark_grey">
     <color rgba="0.3 0.3 0.3 1.0"/>
@@ -14,4 +14,7 @@
     <color rgba="0.2 0.2 0.8 1.0"/>
   </material>
+  <material name="orange">
+    <color rgba="0.9 0.5 0.1 1.0"/>
+  </material>
   <!-- ==================== Properties ==================== -->
   <xacro:property name="chassis_length" value="0.6"/>
@@ -19,8 +22,9 @@
   <xacro:property name="chassis_height" value="0.15"/>
   <xacro:property name="chassis_mass"   value="20.0"/>
+  <xacro:property name="top_plate_height" value="0.005"/>
   <xacro:property name="wheel_radius" value="0.075"/>
-  <xacro:property name="wheel_width"  value="0.03"/>
+  <xacro:property name="wheel_width"  value="0.05"/>
   <xacro:property name="wheel_mass"   value="1.0"/>
-  <xacro:property name="caster_radius" value="0.025"/>
+  <xacro:property name="caster_radius" value="0.04"/>
   <xacro:property name="caster_mass"   value="0.3"/>
   <!-- ==================== Inertia Macros ==================== -->
@@ -68,8 +72,13 @@
       <parent link="base_link"/>
       <child link="${prefix}_wheel_link"/>
-      <origin xyz="0 ${y_reflect * (chassis_width/2.0 + wheel_width/2.0)} 0" rpy="${-pi/2.0} 0 0"/>
+      <origin xyz="0 ${y_reflect * (chassis_width/2.0 + wheel_width/2.0)} ${-chassis_height/2.0}" rpy="${-pi/2.0} 0 0"/>
       <axis xyz="0 0 1"/>
       <dynamics damping="0.01" friction="0.1"/>
     </joint>
+    <gazebo reference="${prefix}_wheel_link">
+      <material>Gazebo/FlatBlack</material>
+      <mu1>1.0</mu1>
+      <mu2>1.0</mu2>
+    </gazebo>
   </xacro:macro>
   <!-- ==================== Caster Macro ==================== -->
@@ -92,7 +101,8 @@
       <parent link="base_link"/>
       <child link="${prefix}_caster_link"/>
-      <origin xyz="${x_offset} 0 ${-(chassis_height/2.0 + caster_radius)}" rpy="0 0 0"/>
+      <origin xyz="${x_offset} 0 ${-(wheel_radius + chassis_height/2.0 - caster_radius)}" rpy="0 0 0"/>
     </joint>
     <gazebo reference="${prefix}_caster_link">
+      <material>Gazebo/Grey</material>
       <mu1>0.001</mu1>
       <mu2>0.001</mu2>
@@ -106,5 +116,4 @@
     <parent link="base_footprint"/>
     <child link="base_link"/>
-    <!-- Place base_link at the centre of the chassis; wheels touch the ground at z=0 -->
     <origin xyz="0 0 ${wheel_radius + chassis_height/2.0}" rpy="0 0 0"/>
   </joint>
@@ -124,4 +133,53 @@
     <xacro:box_inertia m="${chassis_mass}" x="${chassis_length}" y="${chassis_width}" z="${chassis_height}"/>
   </link>
+  <gazebo reference="base_link">
+    <material>Gazebo/FlatBlack</material>
+  </gazebo>
+  <!-- ==================== Top Cover Plate ==================== -->
+  <link name="top_plate_link">
+    <visual>
+      <geometry>
+        <box size="${chassis_length - 0.02} ${chassis_width - 0.02} ${top_plate_height}"/>
+      </geometry>
+      <material name="orange"/>
+    </visual>
+    <collision>
+      <geometry>
+        <box size="${chassis_length - 0.02} ${chassis_width - 0.02} ${top_plate_height}"/>
+      </geometry>
+    </collision>
+    <xacro:box_inertia m="0.5" x="${chassis_length - 0.02}" y="${chassis_width - 0.02}" z="${top_plate_height}"/>
+  </link>
+  <joint name="top_plate_joint" type="fixed">
+    <parent link="base_link"/>
+    <child link="top_plate_link"/>
+    <origin xyz="0 0 ${chassis_height/2.0 + top_plate_height/2.0}" rpy="0 0 0"/>
+  </joint>
+  <gazebo reference="top_plate_link">
+    <material>Gazebo/Orange</material>
+  </gazebo>
+  <!-- ==================== Front Bumper (visual indicator of forward direction) ==================== -->
+  <link name="front_bumper_link">
+    <visual>
+      <geometry>
+        <box size="0.02 ${chassis_width + 0.02} 0.06"/>
+      </geometry>
+      <material name="orange"/>
+    </visual>
+    <collision>
+      <geometry>
+        <box size="0.02 ${chassis_width + 0.02} 0.06"/>
+      </geometry>
+    </collision>
+    <xacro:box_inertia m="0.2" x="0.02" y="${chassis_width + 0.02}" z="0.06"/>
+  </link>
+  <joint name="front_bumper_joint" type="fixed">
+    <parent link="base_link"/>
+    <child link="front_bumper_link"/>
+    <origin xyz="${chassis_length/2.0} 0 0" rpy="0 0 0"/>
+  </joint>
+  <gazebo reference="front_bumper_link">
+    <material>Gazebo/Orange</material>
+  </gazebo>
   <!-- ==================== Drive Wheels ==================== -->
   <xacro:drive_wheel prefix="left"  y_reflect="1"/>
@@ -130,4 +188,27 @@
   <xacro:caster_wheel prefix="front" x_offset="${chassis_length/2.0 - caster_radius - 0.02}"/>
   <xacro:caster_wheel prefix="rear"  x_offset="${-(chassis_length/2.0 - caster_radius - 0.02)}"/>
+  <!-- ==================== Sensor Tower (raises LiDAR above chassis) ==================== -->
+  <link name="sensor_tower_link">
+    <visual>
+      <geometry>
+        <cylinder radius="0.03" length="0.15"/>
+      </geometry>
+      <material name="dark_grey"/>
+    </visual>
+    <collision>
+      <geometry>
+        <cylinder radius="0.03" length="0.15"/>
+      </geometry>
+    </collision>
+    <xacro:cylinder_inertia m="0.3" r="0.03" h="0.15"/>
+  </link>
+  <joint name="sensor_tower_joint" type="fixed">
+    <parent link="base_link"/>
+    <child link="sensor_tower_link"/>
+    <origin xyz="0 0 ${chassis_height/2.0 + 0.075}" rpy="0 0 0"/>
+  </joint>
+  <gazebo reference="sensor_tower_link">
+    <material>Gazebo/FlatBlack</material>
+  </gazebo>
   <!-- ==================== Velodyne VLP-16 LiDAR ==================== -->
   <link name="velodyne_link">
@@ -148,8 +229,8 @@
     <parent link="base_link"/>
     <child link="velodyne_link"/>
-    <!-- z=0.25m above base_link centre -->
-    <origin xyz="0 0 0.25" rpy="0 0 0"/>
+    <origin xyz="0 0 ${chassis_height/2.0 + 0.15 + 0.035}" rpy="0 0 0"/>
   </joint>
   <gazebo reference="velodyne_link">
+    <material>Gazebo/Blue</material>
     <sensor name="velodyne" type="gpu_ray">
       <always_on>true</always_on>
@@ -209,5 +290,5 @@
     <parent link="base_link"/>
     <child link="camera_link"/>
-    <origin xyz="0.3 0 0.15" rpy="0 0 0"/>
+    <origin xyz="${chassis_length/2.0 - 0.01} 0 ${chassis_height/2.0 + 0.02}" rpy="0 0 0"/>
   </joint>
   <!-- Optical frame (ROS convention: z forward, x right, y down) -->
@@ -219,4 +300,5 @@
   </joint>
   <gazebo reference="camera_link">
+    <material>Gazebo/White</material>
     <sensor name="realsense_d435" type="depth">
       <always_on>true</always_on>
@@ -310,5 +392,5 @@
       <left_joint>left_wheel_joint</left_joint>
       <right_joint>right_wheel_joint</right_joint>
-      <wheel_separation>0.4</wheel_separation>
+      <wheel_separation>0.45</wheel_separation>
       <wheel_diameter>0.15</wheel_diameter>
       <max_wheel_torque>10.0</max_wheel_torque>
